File: PCB.sch (KiCad schematic (older format))
At the start: 27 parts, among them J1 Conn_01x03_Male, J2 Conn_01x04_Male, J3 Conn_02x03_Odd_Even, J4 Conn_01x03_Male, U1 L7805, U2 TMA1215D, U3 ATTINY2313-20PU, U4 DAC0808_DIP, U5 LM358, U6 DS18B20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

Commit message: PCB erstellt
Parts:
- added C8, C9: C, Capacitors_THT:C_Disc_D3.8mm_W2.6mm_P2.50mm, symbol C
Connections:
- net +15V: now also C9.1
- net -15V: now also C8.1
- net GND: now also C8.2, C9.2
Changed lines of the file:
@@
 LIBS:maxim
 LIBS:tracco
+LIBS:PCB-cache
 EELAYER 25 0
 EELAYER END
@@
 OneWire
 $Comp
-L -15V #PWR16
+L -15V #PWR19
 U 1 1 5A5A29EB
 P 6850 2050
-F 0 "#PWR16" H 6850 2150 50  0001 C CNN
+F 0 "#PWR19" H 6850 2150 50  0001 C CNN
 F 1 "-15V" H 6850 2200 50  0000 C CNN
 F 2 "" H 6850 2050 50  0001 C CNN
@@
 $EndComp
 $Comp
-L -15V #PWR23
+L -15V #PWR26
 U 1 1 5A5A318D
 P 8050 1700
-F 0 "#PWR23" H 8050 1800 50  0001 C CNN
+F 0 "#PWR26" H 8050 1800 50  0001 C CNN
 F 1 "-15V" H 8050 1850 50  0000 C CNN
 F 2 "" H 8050 1700 50  0001 C CNN
@@
 Wire Wire Line
 	7450 3900 7450 3950
+$Comp
+L C C8
+U 1 1 5A5AF319
+P 4650 1950
+F 0 "C8" H 4675 2050 50  0000 L CNN
+F 1 "C" H 4675 1850 50  0000 L CNN
+F 2 "Capacitors_THT:C_Disc_D3.8mm_W2.6mm_P2.50mm" H 4688 1800 50  0001 C CNN
+F 3 "" H 4650 1950 50  0001 C CNN
+	1    4650 1950
+	1    0    0    -1
+$EndComp
+$Comp
+L C C9
+U 1 1 5A5AF3B0
+P 4900 1950
+F 0 "C9" H 4925 2050 50  0000 L CNN
+F 1 "C" H 4925 1850 50  0000 L CNN
+F 2 "Capacitors_THT:C_Disc_D3.8mm_W2.6mm_P2.50mm" H 4938 1800 50  0001 C CNN
+F 3 "" H 4900 1950 50  0001 C CNN
+	1    4900 1950
+	1    0    0    -1
+$EndComp
+$Comp
+L GND #PWR026
+U 1 1 5A5AF4A4
+P 4900 2200
+F 0 "#PWR026" H 4900 1950 50  0001 C CNN
+F 1 "GND" H 4900 2050 50  0000 C CNN
+F 2 "" H 4900 2200 50  0001 C CNN
+F 3 "" H 4900 2200 50  0001 C CNN
+	1    4900 2200
+	1    0    0    -1
+$EndComp
+$Comp
+L -15V #PWR10
+U 1 1 5A5AF506
+P 4650 1700
+F 0 "#PWR10" H 4650 1800 50  0001 C CNN
+F 1 "-15V" H 4650 1850 50  0000 C CNN
+F 2 "" H 4650 1700 50  0001 C CNN
+F 3 "" H 4650 1700 50  0001 C CNN
+	1    4650 1700
+	1    0    0    -1
+$EndComp
+$Comp
+L +15V #PWR027
+U 1 1 5A5AF568
+P 4900 1700
+F 0 "#PWR027" H 4900 1550 50  0001 C CNN
+F 1 "+15V" H 4900 1840 50  0000 C CNN
+F 2 "" H 4900 1700 50  0001 C CNN
+F 3 "" H 4900 1700 50  0001 C CNN
+	1    4900 1700
+	1    0    0    -1
+$EndComp
+Wire Wire Line
+	4650 2100 4650 2150
+Wire Wire Line
+	4650 2150 4900 2150
+Wire Wire Line
+	4900 2100 4900 2200
+Connection ~ 4900 2150
+Wire Wire Line
+	4650 1800 4650 1700
+Wire Wire Line
+	4900 1800 4900 1700
 $EndSCHEMATC
