File: PCB/PCB.kicad_pcb (KiCad board)
At the start: 2 copper layers, 29 parts, among them J1 Conn_01x03_Male, J2 Conn_01x04_Male, J3 Conn_02x03_Odd_Even, J4 Conn_01x03_Male, U1 L7805, U2 TMA1215D, U3 ATTINY2313-20PU, U4 DAC0808_DIP, U5 LM358, U6 DS18B20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

Commit message: add box
Other:
- board outline added: 64.9 x 45.2 mm
Changed lines of the file:
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@@
     (links 78)
     (no_connects 0)
-    (area 93.498999 74.437142 158.596001 123.527)
+    (area 93.472 72.103001 167.044488 123.527)
     (thickness 1.6)
     (drawings 7)
@@
     (38 B.Mask user)
     (39 F.Mask user)
-    (40 Dwgs.User user)
+    (40 Dwgs.User user hide)
     (41 Cmts.User user)
     (42 Eco1.User user)
@@
     (trace_min 0.2)
     (segment_width 0.2)
-    (edge_width 0.15)
+    (edge_width 0.1)
     (via_size 0.6)
     (via_drill 0.4)
@@
     )
   )
+  (gr_line (start 93.599 77.216) (end 93.599 77.343) (angle 90) (layer Edge.Cuts) (width 0.1))
+  (gr_line (start 158.496 77.216) (end 93.599 77.216) (angle 90) (layer Edge.Cuts) (width 0.1))
+  (gr_line (start 158.496 122.428) (end 158.496 77.216) (angle 90) (layer Edge.Cuts) (width 0.1))
   (dimension 45.085179 (width 0.3) (layer Dwgs.User)
     (gr_text "45,085 mm" (at 160.544488 99.891092 89.83860386) (layer Dwgs.User)
@@
     (arrow2b (pts (xy 158.623 74.803001) (xy 157.496496 75.389422)))
   )
-  (gr_line (start 158.496 77.343) (end 158.242 77.343) (angle 90) (layer Margin) (width 0.2))
-  (gr_line (start 158.496 122.428) (end 158.496 77.343) (angle 90) (layer Margin) (width 0.2))
-  (gr_line (start 93.599 122.428) (end 158.496 122.428) (angle 90) (layer Margin) (width 0.2))
-  (gr_line (start 93.599 77.343) (end 93.599 122.428) (angle 90) (layer Margin) (width 0.2))
-  (gr_line (start 158.242 77.343) (end 93.599 77.343) (angle 90) (layer Margin) (width 0.2))
+  (gr_line (start 93.599 122.428) (end 158.496 122.428) (angle 90) (layer Edge.Cuts) (width 0.2))
+  (gr_line (start 93.599 77.343) (end 93.599 122.428) (angle 90) (layer Edge.Cuts) (width 0.1))
   (segment (start 140.462 116.078) (end 141.478 116.078) (width 0.25) (layer B.Cu) (net 1))
   (segment (start 141.478 116.078) (end 142.748 114.808) (width 0.25) (layer B.Cu) (net 1))
